File: pcb/piweather.kicad_pcb (KiCad board)
At the start: 4 copper layers, 35 x 35 mm, 70 parts, among them J1 USB_B_Micro, J3 CONN127P-02X13-M55-7012642R, J5 CONN_01X03, U1 STM32F405RGTx, U2 AP3418, U3 SN65HVD232D, U4 AS5047P, Y1 Crystal_GND24

Commit message: wip
Parts:
- removed C1: CC0603JRNPO8BN102, Main:CAPC0603
- removed C10, C11: CC0805MKX5R5BB226, Main:CAPC0805
- removed C12, C15: CC0603JRNPO9BN100, Main:CAPC0603
- removed C13, C14, C16, C21, C4, C5, C6, C7, C8: CC0603KRX7R7BB104, Main:CAPC0603
- removed C17, C18: CC0603KRX7R9BB222, Main:CAPC0603
- removed C19, C20: CC0603JRNPO9BN470, Main:CAPC0603
- removed C2, C3: CC0603KRX5R5BB225, Main:CAPC0603
- removed C9: CC0603KRX5R5BB475, Main:CAPC0603
- removed D1: MBR0520LT1G, Main:SOD3717X135
- removed D2: SMF, Diode_SMD:D_SOD-123F
- removed D3: LTW-170TK, Main:DIOC200X120X110
- removed FB1: Ferrite_Bead, Capacitor_SMD:C_0603_1608Metric
- removed J3: CONN127P-02X13-M55-7012642R, Main:CONN127P-02X13-M55-7012642R
- removed J5: CONN_01X03, Main:SOCKET254P-01X03
- removed L1: INDUCTOR_SRN4026-2R2Y, Main:INDP400400X250
- removed R1: RC0603FR-0710RL, Main:RESC0603
- removed R11, R12, R13, R5, R6: RC0603FR-0722R1L, Main:RESC0603
- removed R14, R8: RC0603FR-07100KL, Main:RESC0603
- removed R15, R16, R17: RC0603FR-07499RL, Main:RESC0603
- removed R18: RC0603FR-070RL, Main:RESC0603
- removed R2: RC0603FR-0727K4L, Main:RESC0603
- removed R3: RC0603FR-076K04L, Main:RESC0603
- removed R4: RC0603FR-07121RL, Main:RESC0603
- removed R9: RC0603FR-0710KL, Main:RESC0603
- removed TP11, TP12, TP13, TP14, TP15, TP16, TP17, TP18, TP19, TP2, TP3, TP4, TP5, TP6, TP8, TP9: TestPoint, Main:TestPoint000
- removed U1: STM32F405RGTx, Package_QFP:LQFP-64_10x10mm_P0.5mm
- removed U2: AP3418, Main:SOT095P300X150X145-5
- removed U3: SN65HVD232D, Main:SOIC127P490X390X175-8
- removed U4: AS5047P, Package_SO:SSOP-14_5.3x6.2mm_P0.65mm
- removed Y1: Crystal_GND24, Crystal:Crystal_SMD_Abracon_ABM3B-4Pin_5.0x3.2mm
- added J2: Conn_01x08_Male, Main:PICOBLADE_FEMALE_8, F.Cu at (95.4, 68.9)
- H1, H2, H3, H4: footprint Main:MECH_NPTH_M3 -> Main:RPi_Hat_Mounting_Hole
- J1: value USB_B_Micro -> Screw_Terminal_01x10; footprint Connector_USB:USB_Micro-B_Amphenol_10103594-0001LF_Horizontal -> Main:Terminal_block_OSTVN10A150
- moved H2 92.0 mm to (71.0, 111.5)
- moved H1 63.4 mm to (71.0, 88.5)
- moved J1 60.4 mm to (115.2, 68.1), turned to 180 degrees
- moved H4 33.7 mm to (129.0, 88.5)
- moved H3 9.33 mm to (129.0, 111.5)
Connections:
- J1 pad 1: /USB_VBUS -> (no net)
- J1 pad 2: /USB_D_N -> (no net)
- J1 pad 3: /USB_D_P -> (no net)
- J1 pad 5: GND -> (no net)
- J1 pad 6: GND -> (no net)
Routing:
- net GNDA: track 75.3 -> 0.00 mm, vias 6 -> 0
- net GND: track 54.0 -> 0.00 mm, vias 16 -> 0
- net /nFAULT_C: track 46.2 -> 0.00 mm, vias 6 -> 0
- net /GPIO7: track 37.6 -> 0.00 mm, vias 3 -> 0
- net +5V: track 36.4 -> 0.00 mm, vias 11 -> 0
- net /M0_CH: track 33.9 -> 0.00 mm, vias 3 -> 0
- net /I2C1_SCL: track 33.7 -> 0.00 mm, vias 4 -> 0
- net /I2C1_SDA: track 33.4 -> 0.00 mm, vias 5 -> 0
- net /nRST: track 33.1 -> 0.00 mm, vias 3 -> 0
- net /GPIO8: track 32.3 -> 0.00 mm, vias 3 -> 0
- net /M0_AH: track 31.0 -> 0.00 mm, vias 3 -> 0
- net /M0_SO1_C: track 30.6 -> 0.00 mm, vias 3 -> 0
- net /M0_CL: track 29.4 -> 0.00 mm, vias 3 -> 0
- net /M0_BL: track 28.1 -> 0.00 mm, vias 3 -> 0
- net /M0_BH: track 27.0 -> 0.00 mm, vias 3 -> 0
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- removed copper zone on B.Cu, net +3V3
- removed copper zone on F.Cu, net +3V3
- removed copper zone on B.Cu, net +5V
- removed copper zone on In2.Cu, net +5V
- removed copper zone on F.Cu, net GND
- removed copper zone on In1.Cu, net GND
- removed copper zone on In2.Cu, net GND
Other:
- board size 35 x 35 mm -> 65 x 50.5 mm
- board text removed: "3V3"
- board text removed: "5V"
- board text removed: "BOOT0"
- board text removed: "Board center X148.5 Y105"
- board text removed: "DIR"
- board text removed: "GND"
- board text removed: "GPIO5"
- board text removed: "GPIO7"
- board text removed: "GPIO8"
- board text removed: "I2C1_SCL"
- board text removed: "I2C1_SDA"
- board text removed: "RX"
- board text removed: "STEP"
- board text removed: "SWCLK"
- board text removed: "SWDIO"
- board text removed: "TX"
- board text removed: "~RST"

Commit message: wip
Parts:
- added J3: Screw_Terminal_01x02, Main:TerminalBlock_1X2_P5.08mm, F.Cu at (80.6, 69.2)
- added J4: Raspberry_Pi_2_3, Main:RPi_2x20_SMT, F.Cu at (100.0, 88.5)
- added U1: FT2232D, Package_QFP:LQFP-48_7x7mm_P0.5mm, F.Cu at (113.6, 103.7)
- added U2: THVD1500, Main:SOIC127P490X390X175-8, F.Cu at (99.7, 103.8)
- J1: value Screw_Terminal_01x10 -> Screw_Terminal_01x08; footprint Main:Terminal_block_OSTVN10A150 -> Main:Terminal_block_OSTVN08A150

Commit message: wip
Parts:
- added H6: MountingHole, Main:RPi_Hat_Mounting_Hole, F.Cu at (71.0, 60.5)
- added U3: THVD1500, Main:SOIC127P490X390X175-8, F.Cu at (108.1, 103.4)
- added U4: V78E05-1000-SMT-TR, Main:V78E05-1000-SMT-TR, F.Cu at (89.6, 69.3)
- U2: value THVD1500 -> PSK-S5B-5; footprint Main:SOIC127P490X390X175-8 -> Main:PSK-S5B-5
- moved J2 44.6 mm to (127.6, 99.8), turned to 90 degrees
- moved U2 33.0 mm to (97.6, 70.8)
- moved U1 26.7 mm to (87.1, 100.3)
- moved J3 7.58 mm to (73.1, 70.3), turned to 270 degrees
- moved J1 6.95 mm to (121.6, 70.8), turned to 90 degrees
Other:
- board size 65 x 50.5 mm -> 65 x 58 mm

Commit message: wip
Parts:
- added U5: Si7020-A20, Package_DFN_QFN:DFN-6-1EP_3x3mm_P1mm_EP1.5x2.4mm, F.Cu at (109.1, 98.8)
- J1: value Screw_Terminal_01x08 -> Screw_Terminal_01x10; footprint Main:Terminal_block_OSTVN08A150 -> Main:Terminal_block_OSTVN10A150
- J3: value Screw_Terminal_01x02 -> Screw_Terminal_01x03; footprint Main:TerminalBlock_1X2_P5.08mm -> Main:TerminalBlock_1X3_P5.08mm
- moved U3 12.9 mm to (119.8, 98.0)
- moved U4 7.92 mm to (97.5, 69.9)
- moved J3 5.89 mm to (77.2, 74.5)
- moved U2 3.00 mm to (100.6, 70.9)
- moved J1 1.50 mm to (123.1, 70.8)
- moved U1 0.27 mm to (87.3, 100.1)
Other:
- board text added: "-DC"
- board text added: "D+"
- board text added: "D-"
- board text added: "Live +DC"
- board text added: "Neut"
- board text added: "SCL"
- board text added: "SDA"

Commit message: wip
Parts:
- added J10: Conn_01x03_Male, Main:SOCKET254P-01X03-0705530002, F.Cu at (107.0, 101.3)
- added J11: Conn_01x03_Male, Main:SOCKET254P-01X03-0705530002, F.Cu at (81.2, 100.5)
- added J5: Conn_01x03_Male, Main:SOCKET254P-01X03-0705530002, F.Cu at (118.4, 101.3)
- moved U5 30.2 mm to (81.5, 111.0)
- moved U3 27.5 mm to (92.4, 97.0)
- moved U1 9.35 mm to (92.6, 107.8)
- moved U2 0.97 mm to (100.6, 69.9)
Changed lines of the file:
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@@
     (tracks 0)
     (zones 0)
-    (modules 14)
+    (modules 17)
     (nets 1)
   )
@@
   )
   (module Main:PICOBLADE_FEMALE_8 (layer F.Cu)
-    (at 127.6 99.775 90)
+    (at 127.6 99.8 90)
     (fp_text reference J2 (at 0 1.6 90) (layer F.SilkS)
       (effects (font (size 1 1) (thickness 0.15)))
@@
   )
   (module Package_QFP:LQFP-48_7x7mm_P0.5mm (layer F.Cu)
-    (at 87.29 100.085)
+    (at 92.6 107.775)
     (descr "48 LEAD LQFP 7x7mm (see MICREL LQFP7x7-48LD-PL-1.pdf)")
     (tags "QFP 0.5")
@@
   )
   (module Main:PSK-S5B-5 (layer F.Cu)
-    (at 100.6 70.875)
+    (at 100.6 69.9)
     (fp_text reference U2 (at 8 10.975) (layer F.SilkS)
       (effects (font (size 1 1) (thickness 0.15)))
@@
   )
   (module Main:SOIC127P490X390X175-8 (layer F.Cu)
-    (at 119.85 98.025)
+    (at 92.4 96.975)
     (descr "14-Lead Plastic Small Outline (SL) - Narrow, 3.90 mm Body [SOIC] (see Microchip Packaging Specification 00000049BS.pdf)")
     (tags "SOIC 1.27")
@@
   )
   (module Package_DFN_QFN:DFN-6-1EP_3x3mm_P1mm_EP1.5x2.4mm (layer F.Cu)
-    (at 109.1 98.775 180)
+    (at 81.5 110.975 180)
     (descr "DFN, 6 Pin (https://www.silabs.com/documents/public/data-sheets/Si7020-A20.pdf), generated with kicad-footprint-generator ipc_dfn_qfn_generator.py")
     (tags "DFN DFN_QFN")
@@
     )
   )
+  (module Main:SOCKET254P-01X03-0705530002 (layer F.Cu)
+    (at 118.4 101.3)
+    (descr "Through hole socket strip")
+    (tags "socket strip")
+    (fp_text reference J5 (at 0 -2.5) (layer F.SilkS)
+      (effects (font (size 1 1) (thickness 0.15)))
+    )
+    (fp_text value Conn_01x03_Male (at 0 2) (layer F.Fab) hide
+      (effects (font (size 0.127 0.127) (thickness 0.03)))
+    )
+    (fp_line (start -3.81 -1.55) (end -3.81 1.55) (layer F.SilkS) (width 0.15))
+    (fp_line (start -3.81 -1.55) (end -2.26 -1.55) (layer F.SilkS) (width 0.15))
+    (fp_line (start -1.27 1.27) (end -1.27 -1.27) (layer F.SilkS) (width 0.15))
+    (fp_line (start 3.81 -1.27) (end 3.81 1.27) (layer F.SilkS) (width 0.15))
+    (fp_line (start -2.26 1.55) (end -3.81 1.55) (layer F.SilkS) (width 0.15))
+    (fp_line (start -1.27 1.27) (end 3.81 1.27) (layer F.SilkS) (width 0.15))
+    (fp_line (start -1.27 -1.27) (end 3.81 -1.27) (layer F.SilkS) (width 0.15))
+    (fp_line (start -5.5 13.5) (end 5.5 13.5) (layer F.CrtYd) (width 0.05))
+    (fp_line (start -5.5 -1.75) (end 5.5 -1.75) (layer F.CrtYd) (width 0.05))
+    (fp_line (start 5.5 -1.75) (end 5.5 13.5) (layer F.CrtYd) (width 0.05))
+    (fp_line (start -5.5 -1.75) (end -5.5 13.5) (layer F.CrtYd) (width 0.05))
+    (pad 3 thru_hole oval (at 2.54 0) (size 1.7272 2.032) (drill 1.016) (layers *.Cu *.Mask F.SilkS))
+    (pad 2 thru_hole oval (at 0 0) (size 1.7272 2.032) (drill 1.016) (layers *.Cu *.Mask F.SilkS))
+    (pad 1 thru_hole rect (at -2.54 0) (size 1.7272 2.032) (drill 1.016) (layers *.Cu *.Mask F.SilkS))
+    (model ${KISYS3DMOD}/main.3dshapes/SOCKET254P-01X03-0705530002.step
+      (at (xyz 0 0 0))
+      (scale (xyz 1 1 1))
+      (rotate (xyz 0 0 180))
+    )
+  )
+  (module Main:SOCKET254P-01X03-0705530002 (layer F.Cu)
+    (at 107 101.3)
+    (descr "Through hole socket strip")
+    (tags "socket strip")
+    (fp_text reference J10 (at 0 -2.5) (layer F.SilkS)
+      (effects (font (size 1 1) (thickness 0.15)))
+    )
+    (fp_text value Conn_01x03_Male (at 0 2) (layer F.Fab) hide
+      (effects (font (size 0.127 0.127) (thickness 0.03)))
+    )
+    (fp_line (start -5.5 -1.75) (end -5.5 13.5) (layer F.CrtYd) (width 0.05))
+    (fp_line (start 5.5 -1.75) (end 5.5 13.5) (layer F.CrtYd) (width 0.05))
+    (fp_line (start -5.5 -1.75) (end 5.5 -1.75) (layer F.CrtYd) (width 0.05))
+    (fp_line (start -5.5 13.5) (end 5.5 13.5) (layer F.CrtYd) (width 0.05))
+    (fp_line (start -1.27 -1.27) (end 3.81 -1.27) (layer F.SilkS) (width 0.15))
+    (fp_line (start -1.27 1.27) (end 3.81 1.27) (layer F.SilkS) (width 0.15))
+    (fp_line (start -2.26 1.55) (end -3.81 1.55) (layer F.SilkS) (width 0.15))
+    (fp_line (start 3.81 -1.27) (end 3.81 1.27) (layer F.SilkS) (width 0.15))
+    (fp_line (start -1.27 1.27) (end -1.27 -1.27) (layer F.SilkS) (width 0.15))
+    (fp_line (start -3.81 -1.55) (end -2.26 -1.55) (layer F.SilkS) (width 0.15))
+    (fp_line (start -3.81 -1.55) (end -3.81 1.55) (layer F.SilkS) (width 0.15))
+    (pad 1 thru_hole rect (at -2.54 0) (size 1.7272 2.032) (drill 1.016) (layers *.Cu *.Mask F.SilkS))
+    (pad 2 thru_hole oval (at 0 0) (size 1.7272 2.032) (drill 1.016) (layers *.Cu *.Mask F.SilkS))
+    (pad 3 thru_hole oval (at 2.54 0) (size 1.7272 2.032) (drill 1.016) (layers *.Cu *.Mask F.SilkS))
+    (model ${KISYS3DMOD}/main.3dshapes/SOCKET254P-01X03-0705530002.step
+      (at (xyz 0 0 0))
+      (scale (xyz 1 1 1))
+      (rotate (xyz 0 0 180))
+    )
+  )
+  (module Main:SOCKET254P-01X03-0705530002 (layer F.Cu)
+    (at 81.2 100.5 270)
+    (descr "Through hole socket strip")
+    (tags "socket strip")
+    (fp_text reference J11 (at 0 -2.5 270) (layer F.SilkS)
+      (effects (font (size 1 1) (thickness 0.15)))
+    )
+    (fp_text value Conn_01x03_Male (at 0 2 270) (layer F.Fab) hide
+      (effects (font (size 0.127 0.127) (thickness 0.03)))
+    )
+    (fp_line (start -5.5 -1.75) (end -5.5 13.5) (layer F.CrtYd) (width 0.05))
+    (fp_line (start 5.5 -1.75) (end 5.5 13.5) (layer F.CrtYd) (width 0.05))
+    (fp_line (start -5.5 -1.75) (end 5.5 -1.75) (layer F.CrtYd) (width 0.05))
+    (fp_line (start -5.5 13.5) (end 5.5 13.5) (layer F.CrtYd) (width 0.05))
+    (fp_line (start -1.27 -1.27) (end 3.81 -1.27) (layer F.SilkS) (width 0.15))
+    (fp_line (start -1.27 1.27) (end 3.81 1.27) (layer F.SilkS) (width 0.15))
+    (fp_line (start -2.26 1.55) (end -3.81 1.55) (layer F.SilkS) (width 0.15))
+    (fp_line (start 3.81 -1.27) (end 3.81 1.27) (layer F.SilkS) (width 0.15))
+    (fp_line (start -1.27 1.27) (end -1.27 -1.27) (layer F.SilkS) (width 0.15))
+    (fp_line (start -3.81 -1.55) (end -2.26 -1.55) (layer F.SilkS) (width 0.15))
+    (fp_line (start -3.81 -1.55) (end -3.81 1.55) (layer F.SilkS) (width 0.15))
+    (pad 1 thru_hole rect (at -2.54 0 270) (size 1.7272 2.032) (drill 1.016) (layers *.Cu *.Mask F.SilkS))
+    (pad 2 thru_hole oval (at 0 0 270) (size 1.7272 2.032) (drill 1.016) (layers *.Cu *.Mask F.SilkS))
+    (pad 3 thru_hole oval (at 2.54 0 270) (size 1.7272 2.032) (drill 1.016) (layers *.Cu *.Mask F.SilkS))
+    (model ${KISYS3DMOD}/main.3dshapes/SOCKET254P-01X03-0705530002.step
+      (at (xyz 0 0 0))
+      (scale (xyz 1 1 1))
+      (rotate (xyz 0 0 180))
+    )
+  )

Commit message: wip
Parts:
- removed J3: Screw_Terminal_01x03, Main:TerminalBlock_1X3_P5.08mm
- added J12: Conn_01x02_Male, Main:AC_terminal_4300.0104, F.Cu at (70.5, 71.5)
- added J6: Conn_01x01_Male, Connector_PinHeader_1.00mm:PinHeader_1x01_P1.00mm_Vertical, F.Cu at (99.6, 113.3)
- moved U5 57.6 mm to (87.3, 53.7)
- moved U3 43.7 mm to (102.1, 54.4)
- moved H6 6.00 mm to (71.0, 54.5)
- moved J11 4.20 mm to (77.0, 100.5)
- moved J1 2.99 mm to (122.0, 68.0)
- moved U2 2.10 mm to (98.5, 69.8)
Other:
- board size 65 x 58 mm -> 65 x 64 mm
- board text removed: "-DC"
- board text removed: "Live +DC"
- board text removed: "Neut"

Commit message: wip, needs routing
Parts:
- added J3: Screw_Terminal_01x02, Main:TerminalBlock_1X2_P5.08mm, F.Cu at (73.1, 69.0)
- added J7: Conn_01x01_Male, Main:POGOPIN_5mm_P70-2300045R, F.Cu at (121.2, 108.5)
- added J8: Conn_01x01_Male, Main:POGOPIN_5mm_P70-2300045R, F.Cu at (109.5, 113.2)
- added J9: Conn_01x01_Male, Main:POGOPIN_5mm_P70-2300045R, F.Cu at (107.7, 113.2)
- J6: footprint Connector_PinHeader_1.00mm:PinHeader_1x01_P1.00mm_Vertical -> Main:POGOPIN_5mm_P70-2300045R
- moved U3 44.0 mm to (95.1, 97.8)
- moved U1 22.3 mm to (113.6, 100.3)
- moved J6 22.1 mm to (121.6, 111.4)
- moved J10 21.3 mm to (86.0, 105.0)
- moved J5 19.7 mm to (99.0, 105.0)
Other:
- board text added: "0V"
- board text added: "DC+"
