File: pcb/piweather.sch (KiCad schematic (older format))
At the start: 61 parts, among them J1 USB_B_Micro, J3 CONN127P-02X13-M55-7012642R, J5 CONN_01X03, U1 STM32F405RGTx, U3 SN65HVD232D, U4 AS5047P, Y1 Crystal_GND24

Commit message: wip
Parts:
- removed C1: CC0603JRNPO8BN102, Main:CAPC0603, symbol cap_smd:CC0603JRNPO8BN102
- removed C12, C15: CC0603JRNPO9BN100, Main:CAPC0603, symbol cap_smd:CC0603JRNPO9BN100
- removed C13, C14, C16, C21, C4, C5, C6, C7, C8: CC0603KRX7R7BB104, Main:CAPC0603, symbol cap_smd:CC0603KRX7R7BB104
- removed C17, C18: CC0603KRX7R9BB222, Main:CAPC0603, symbol cap_smd:CC0603KRX7R9BB222
- removed C19, C20: CC0603JRNPO9BN470, Main:CAPC0603, symbol cap_smd:CC0603JRNPO9BN470
- removed C2, C3: CC0603KRX5R5BB225, Main:CAPC0603, symbol cap_smd:CC0603KRX5R5BB225
- removed D1: MBR0520LT1G, Main:SOD3717X135, symbol devices:MBR0520LT1G
- removed D3: LTW-170TK, Main:DIOC200X120X110, symbol devices:LTW-170TK
- removed FB1: Ferrite_Bead, Capacitor_SMD:C_0603_1608Metric, symbol Device:Ferrite_Bead
- removed J1: USB_B_Micro, Connector_USB:USB_Micro-B_Amphenol_10103594-0001LF_Horizontal, symbol Connector:USB_B_Micro
- removed J3: CONN127P-02X13-M55-7012642R, Main:CONN127P-02X13-M55-7012642R, symbol connect:CONN127P-02X13-M55-7012642R
- removed J5: CONN_01X03, Main:SOCKET254P-01X03, symbol connect:CONN_01X03
- removed R11, R12, R13, R5, R6: RC0603FR-0722R1L, Main:RESC0603, symbol res_smd:RC0603FR-0722R1L
- removed R14, R8: RC0603FR-07100KL, Main:RESC0603, symbol res_smd:RC0603FR-07100KL
- removed R15, R16, R17: RC0603FR-07499RL, Main:RESC0603, symbol res_smd:RC0603FR-07499RL
- removed R18: RC0603FR-070RL, Main:RESC0603, symbol res_smd:RC0603FR-070RL
- removed R4: RC0603FR-07121RL, Main:RESC0603, symbol res_smd:RC0603FR-07121RL
- removed R9: RC0603FR-0710KL, Main:RESC0603, symbol res_smd:RC0603FR-0710KL
- removed TP11, TP12, TP13, TP14, TP15, TP16, TP17, TP18, TP19, TP2, TP3, TP4, TP5, TP6, TP8, TP9: TestPoint, Main:TestPoint000, symbol Connector:TestPoint
- removed U1: STM32F405RGTx, Package_QFP:LQFP-64_10x10mm_P0.5mm, symbol MCU_ST_STM32F4:STM32F405RGTx
- removed U3: SN65HVD232D, Main:SOIC127P490X390X175-8, symbol analog:SN65HVD232D
- removed U4: AS5047P, Package_SO:SSOP-14_5.3x6.2mm_P0.65mm, symbol analog:AS5047P
- removed Y1: Crystal_GND24, Crystal:Crystal_SMD_Abracon_ABM3B-4Pin_5.0x3.2mm, symbol Device:Crystal_GND24
- added J1: Screw_Terminal_01x10, Main:Terminal_block_OSTVN10A150, symbol Connector:Screw_Terminal_01x10
- added J2: Conn_01x08_Male, Main:PICOBLADE_FEMALE_8, symbol Connector:Conn_01x08_Male
- H1, H2, H3, H4: footprint Main:MECH_NPTH_M3 -> Main:RPi_Hat_Mounting_Hole
Connections:
- net labels removed: +3V3, +5V, +VDC, AUX_H, AUX_L, BOOT0, CAN_D, CAN_H, CAN_L, CAN_R, C_SWCLK, C_SWDIO, EN_GATE, GND, GNDA, GPIO1_TX, GPIO2_RX, GPIO3_STEP, GPIO4_DIR, GPIO5, GPIO6, GPIO7, GPIO8, I2C1_SCL, I2C1_SDA, LEDA, M0_AH, M0_AL, M0_BH, M0_BL, M0_CH, M0_CL, M0_ENC_A, M0_ENC_B, M0_ENC_Z, M0_SO1, M0_SO1_C, M0_SO2, M0_SO2_C, M0_TEMP, M0_TEMP_C, M0_nCS, PH0, PH1, SPI_MISO, SPI_MISO_C, SPI_MOSI, SPI_SCK, SWCLK, SWDIO, USB_D_N, USB_D_P, USB_VBUS, VBUS_S, VCAP_1, VCAP_2, VDDA, nFAULT, nFAULT_C, nRST
- wire segments 279 -> 0
- no-connect marks 18 -> 0
Other:
- note removed: "ADD MECHANICAL\nMOUNTING HOLES"
- note removed: "No extra pins for 3.3V\nUse LDO on motor module"
- note removed: "Place 0Ohm near\nMCU"

Commit message: wip
Parts:
- removed J1: Screw_Terminal_01x10, Main:Terminal_block_OSTVN10A150, symbol Connector:Screw_Terminal_01x10
- added J1: Screw_Terminal_01x08, Main:Terminal_block_OSTVN08A150, symbol Connector:Screw_Terminal_01x08
- added J3: Screw_Terminal_01x02, Main:TerminalBlock_1X2_P5.08mm, symbol Connector:Screw_Terminal_01x02
- added J4: Raspberry_Pi_2_3, Main:RPi_2x20_SMT, symbol Connector:Raspberry_Pi_2_3
- added U1: FT2232D, Package_QFP:LQFP-48_7x7mm_P0.5mm, symbol Interface_USB:FT2232D
- added U?: THVD1500, Main:SOIC127P490X390X175-8, symbol analog:THVD1500
Other:
- moved on the sheet: J2
Changed lines of the file:
@@
-$EndComp
-$Comp
-L Connector:Screw_Terminal_01x10 J1
-U 1 1 5D9BBCFA
-P 14500 1850
-F 0 "J1" H 14580 1842 50  0000 L CNN
-F 1 "Screw_Terminal_01x10" H 14580 1751 50  0000 L CNN
-F 2 "Main:Terminal_block_OSTVN10A150" H 14500 1850 50  0001 C CNN
-F 3 "~" H 14500 1850 50  0001 C CNN
-F 4 "On Shore Technology Inc." H 14500 1850 50  0001 C CNN "Manufacturer"
-F 5 "OSTVN10A150" H 14500 1850 50  0001 C CNN "MPN"
-	1    14500 1850
-	1    0    0    -1
 $EndComp
 $Comp
 L Connector:Conn_01x08_Male J2
 U 1 1 5D9BE108
-P 14500 3350
-F 0 "J2" H 14473 3323 50  0000 R CNN
-F 1 "Conn_01x08_Male" H 14473 3232 50  0000 R CNN
-F 2 "Main:PICOBLADE_FEMALE_8" H 14500 3350 50  0001 C CNN
-F 3 "~" H 14500 3350 50  0001 C CNN
-F 4 "Molex" H 14500 3350 50  0001 C CNN "Manufacturer"
-F 5 "0530480810" H 14500 3350 50  0001 C CNN "MPN"
-	1    14500 3350
+P 15050 3100
+F 0 "J2" H 15023 3073 50  0000 R CNN
+F 1 "Conn_01x08_Male" H 15023 2982 50  0000 R CNN
+F 2 "Main:PICOBLADE_FEMALE_8" H 15050 3100 50  0001 C CNN
+F 3 "~" H 15050 3100 50  0001 C CNN
+F 4 "Molex" H 15050 3100 50  0001 C CNN "Manufacturer"
+F 5 "0530480810" H 15050 3100 50  0001 C CNN "MPN"
+	1    15050 3100
 	-1   0    0    -1
 $EndComp
+$Comp
+L Connector:Screw_Terminal_01x02 J3
+U 1 1 5D9CB81D
+P 15050 1100
+F 0 "J3" H 15130 1092 50  0000 L CNN
+F 1 "Screw_Terminal_01x02" H 15130 1001 50  0000 L CNN
+F 2 "Main:TerminalBlock_1X2_P5.08mm" H 15050 1100 50  0001 C CNN
+F 3 "~" H 15050 1100 50  0001 C CNN
+F 4 "Phoenix Contact" H 15050 1100 50  0001 C CNN "Manufacturer"
+F 5 "1715721" H 15050 1100 50  0001 C CNN "MPN"
+	1    15050 1100
+	1    0    0    -1
+$EndComp
+$Comp
+L Connector:Screw_Terminal_01x08 J1
+U 1 1 5D9CBBE8
+P 15050 1850
+F 0 "J1" H 15130 1842 50  0000 L CNN
+F 1 "Screw_Terminal_01x08" H 15130 1751 50  0000 L CNN
+F 2 "Main:Terminal_block_OSTVN08A150" H 15050 1850 50  0001 C CNN
+F 3 "~" H 15050 1850 50  0001 C CNN
+F 4 "On Shore Technology Inc." H 15050 1850 50  0001 C CNN "Manufacturer"
+F 5 "OSTVN08A150" H 15050 1850 50  0001 C CNN "MPN"
+	1    15050 1850
+	1    0    0    -1
+$EndComp
+$Comp
+L Connector:Raspberry_Pi_2_3 J4
+U 1 1 5D9CE7F8
+P 11200 5600
+F 0 "J4" H 11200 7078 50  0000 C CNN
+F 1 "Raspberry_Pi_2_3" H 11200 6987 50  0000 C CNN
+F 2 "Main:RPi_2x20_SMT" H 11200 5600 50  0001 C CNN
+F 3 "https://www.raspberrypi.org/documentation/hardware/raspberrypi/schematics/rpi_SCH_3bplus_1p0_reduced.pdf" H 11200 5600 50  0001 C CNN
+F 4 "Harwin Inc." H 11200 5600 50  0001 C CNN "Manufacturer"
+F 5 "M20-7812045R" H 11200 5600 50  0001 C CNN "MPN"
+	1    11200 5600
+	1    0    0    -1
+$EndComp
+$Comp
+L Interface_USB:FT2232D U1
+U 1 1 5D9CF0E5
+P 4500 4900
+F 0 "U1" H 4500 6978 50  0000 C CNN
+F 1 "FT2232D" H 4500 6887 50  0000 C CNN
+F 2 "Package_QFP:LQFP-48_7x7mm_P0.5mm" H 4500 4900 50  0001 C CNN
+F 3 "http://www.ftdichip.com/Support/Documents/DataSheets/ICs/DS_FT2232D.pdf" H 4500 4900 50  0001 C CNN
+	1    4500 4900
+	1    0    0    -1
+$EndComp
+$Comp
+L analog:THVD1500 U?
+U 1 1 5D9D349A
+P 7950 5350
+F 0 "U?" H 7950 6039 60  0000 C CNN
+F 1 "THVD1500" H 7950 5933 60  0000 C CNN
+F 2 "Main:SOIC127P490X390X175-8" H 8150 4700 60  0001 C CNN
+F 3 "" H 7850 5350 60  0001 C CNN
+F 4 "Texas Instruments" H 7850 4500 60  0001 C CNN "Manufacturer"
+F 5 "THVD1500DR" H 7700 4600 60  0001 C CNN "MPN"
+	1    7950 5350
+	1    0    0    -1
+$EndComp
 $EndSCHEMATC

Commit message: wip
Parts:
- added H6: MountingHole, Main:RPi_Hat_Mounting_Hole, symbol Mechanical:MountingHole
- added U2: PSK-S5B-5, Main:PSK-S5B-5, symbol analog:PSK-S5B-5
- added U4: V78E05-1000-SMT-TR, Main:V78E05-1000-SMT-TR, symbol analog:V78E05-1000-SMT-TR
- gave numbers to parts that had none: 1
Other:
- moved on the sheet: U3
Changed lines of the file:
@@
 $EndComp
 $Comp
-L analog:THVD1500 U?
+L analog:THVD1500 U3
 U 1 1 5D9D349A
-P 7950 5350
-F 0 "U?" H 7950 6039 60  0000 C CNN
-F 1 "THVD1500" H 7950 5933 60  0000 C CNN
-F 2 "Main:SOIC127P490X390X175-8" H 8150 4700 60  0001 C CNN
-F 3 "" H 7850 5350 60  0001 C CNN
-F 4 "Texas Instruments" H 7850 4500 60  0001 C CNN "Manufacturer"
-F 5 "THVD1500DR" H 7700 4600 60  0001 C CNN "MPN"
-	1    7950 5350
+P 8000 5300
+F 0 "U3" H 8000 5989 60  0000 C CNN
+F 1 "THVD1500" H 8000 5883 60  0000 C CNN
+F 2 "Main:SOIC127P490X390X175-8" H 8200 4650 60  0001 C CNN
+F 3 "" H 7900 5300 60  0001 C CNN
+F 4 "Texas Instruments" H 7900 4450 60  0001 C CNN "Manufacturer"
+F 5 "THVD1500DR" H 7750 4550 60  0001 C CNN "MPN"
+	1    8000 5300
 	1    0    0    -1
 $EndComp
+$Comp
+L analog:PSK-S5B-5 U2
+U 1 1 5D9D3E1B
+P 8000 3750
+F 0 "U2" H 8000 4287 60  0000 C CNN
+F 1 "PSK-S5B-5" H 8000 4181 60  0000 C CNN
+F 2 "Main:PSK-S5B-5" H 7900 3150 60  0001 L CNN
+F 3 "" H 8000 3750 60  0001 C CNN
+F 4 "CUI Inc." H 7900 3250 60  0001 L CNN "Manufacturer"
+F 5 "PSK-S5B-5" H 7900 3350 60  0001 L CNN "MPN"
+	1    8000 3750
+	1    0    0    -1
+$EndComp
+$Comp
+L Mechanical:MountingHole H6
+U 1 1 5D9D426D
+P 800 2300
+F 0 "H6" H 900 2346 50  0000 L CNN
+F 1 "MountingHole" H 900 2255 50  0000 L CNN
+F 2 "Main:RPi_Hat_Mounting_Hole" H 800 2300 50  0001 C CNN
+F 3 "~" H 800 2300 50  0001 C CNN
+	1    800  2300
+	1    0    0    -1
+$EndComp
+$Comp
+L analog:V78E05-1000-SMT-TR U4
+U 1 1 5D9D532D
+P 8000 2650
+F 0 "U4" H 8000 3187 60  0000 C CNN
+F 1 "V78E05-1000-SMT-TR" H 8000 3081 60  0000 C CNN
+F 2 "Main:V78E05-1000-SMT-TR" H 7550 2100 60  0001 C CNN
+F 3 "" H 7650 2200 60  0001 C CNN
+F 4 "CUI Inc. " H 8400 2150 60  0001 L CNN "Manufacturer"
+F 5 "V78E05-1000-SMT-TR" H 8400 2250 60  0001 L CNN "MPN"
+	1    8000 2650
+	1    0    0    -1
+$EndComp

Commit message: wip
Other:
- moved on the sheet: J2
Changed lines of the file:
@@
 L Connector:Conn_01x08_Male J2
 U 1 1 5D9BE108
-P 15050 3100
-F 0 "J2" H 15023 3073 50  0000 R CNN
-F 1 "Conn_01x08_Male" H 15023 2982 50  0000 R CNN
-F 2 "Main:PICOBLADE_FEMALE_8" H 15050 3100 50  0001 C CNN
-F 3 "~" H 15050 3100 50  0001 C CNN
-F 4 "Molex" H 15050 3100 50  0001 C CNN "Manufacturer"
-F 5 "0530480810" H 15050 3100 50  0001 C CNN "MPN"
-	1    15050 3100
+P 15050 2850
+F 0 "J2" H 15023 2823 50  0000 R CNN
+F 1 "Conn_01x08_Male" H 15023 2732 50  0000 R CNN
+F 2 "Main:PICOBLADE_FEMALE_8" H 15050 2850 50  0001 C CNN
+F 3 "~" H 15050 2850 50  0001 C CNN
+F 4 "Molex" H 15050 2850 50  0001 C CNN "Manufacturer"
+F 5 "0530480810" H 15050 2850 50  0001 C CNN "MPN"
+	1    15050 2850
 	-1   0    0    -1
 $EndComp
@@
 F 5 "1715721" H 15050 1100 50  0001 C CNN "MPN"
 	1    15050 1100
-	1    0    0    -1
-$EndComp
-$Comp
-L Connector:Screw_Terminal_01x08 J1
-U 1 1 5D9CBBE8
-P 15050 1850
-F 0 "J1" H 15130 1842 50  0000 L CNN
-F 1 "Screw_Terminal_01x08" H 15130 1751 50  0000 L CNN
-F 2 "Main:Terminal_block_OSTVN08A150" H 15050 1850 50  0001 C CNN
-F 3 "~" H 15050 1850 50  0001 C CNN
-F 4 "On Shore Technology Inc." H 15050 1850 50  0001 C CNN "Manufacturer"
-F 5 "OSTVN08A150" H 15050 1850 50  0001 C CNN "MPN"
-	1    15050 1850
 	1    0    0    -1
 $EndComp
@@
 	1    0    0    -1
 $EndComp
+$Comp
+L Connector:Screw_Terminal_01x08 J1
+U 1 1 5D9E30DD
+P 15050 1800
+F 0 "J1" H 15130 1792 50  0000 L CNN
+F 1 "Screw_Terminal_01x08" H 15130 1701 50  0000 L CNN
+F 2 "Main:Terminal_block_OSTVN08A150" H 15050 1800 50  0001 C CNN
+F 3 "~" H 15050 1800 50  0001 C CNN
+F 4 "On Shore Technology Inc." H 15050 1800 50  0001 C CNN "Manufacturer"
+F 5 "OSTVN08A150" H 15050 1800 50  0001 C CNN "MPN"
+	1    15050 1800
+	1    0    0    -1
+$EndComp

Commit message: wip
Parts:
- removed J1: Screw_Terminal_01x08, Main:Terminal_block_OSTVN08A150, symbol Connector:Screw_Terminal_01x08
- removed J3: Screw_Terminal_01x02, Main:TerminalBlock_1X2_P5.08mm, symbol Connector:Screw_Terminal_01x02
- added J1: Screw_Terminal_01x10, Main:Terminal_block_OSTVN10A150, symbol Connector:Screw_Terminal_01x10
- added J3: Screw_Terminal_01x03, Main:TerminalBlock_1X3_P5.08mm, symbol Connector:Screw_Terminal_01x03
- added J? (x2): Conn_01x01_Male, symbol Connector:Conn_01x01_Male
- added U5: Si7020-A20, Package_DFN_QFN:DFN-6-1EP_3x3mm_P1mm_EP1.5x2.4mm, symbol Sensor_Humidity:Si7020-A20
Other:
- moved on the sheet: J2
Changed lines of the file:
@@
 L Connector:Conn_01x08_Male J2
 U 1 1 5D9BE108
-P 15050 2850
-F 0 "J2" H 15023 2823 50  0000 R CNN
-F 1 "Conn_01x08_Male" H 15023 2732 50  0000 R CNN
-F 2 "Main:PICOBLADE_FEMALE_8" H 15050 2850 50  0001 C CNN
-F 3 "~" H 15050 2850 50  0001 C CNN
-F 4 "Molex" H 15050 2850 50  0001 C CNN "Manufacturer"
-F 5 "0530480810" H 15050 2850 50  0001 C CNN "MPN"
-	1    15050 2850
+P 15050 3250
+F 0 "J2" H 15023 3223 50  0000 R CNN
+F 1 "Conn_01x08_Male" H 15023 3132 50  0000 R CNN
+F 2 "Main:PICOBLADE_FEMALE_8" H 15050 3250 50  0001 C CNN
+F 3 "~" H 15050 3250 50  0001 C CNN
+F 4 "Molex" H 15050 3250 50  0001 C CNN "Manufacturer"
+F 5 "0530480810" H 15050 3250 50  0001 C CNN "MPN"
+	1    15050 3250
 	-1   0    0    -1
-$EndComp
-$Comp
-L Connector:Screw_Terminal_01x02 J3
-U 1 1 5D9CB81D
-P 15050 1100
-F 0 "J3" H 15130 1092 50  0000 L CNN
-F 1 "Screw_Terminal_01x02" H 15130 1001 50  0000 L CNN
-F 2 "Main:TerminalBlock_1X2_P5.08mm" H 15050 1100 50  0001 C CNN
-F 3 "~" H 15050 1100 50  0001 C CNN
-F 4 "Phoenix Contact" H 15050 1100 50  0001 C CNN "Manufacturer"
-F 5 "1715721" H 15050 1100 50  0001 C CNN "MPN"
-	1    15050 1100
-	1    0    0    -1
 $EndComp
 $Comp
@@
 $EndComp
 $Comp
-L Connector:Screw_Terminal_01x08 J1
-U 1 1 5D9E30DD
-P 15050 1800
-F 0 "J1" H 15130 1792 50  0000 L CNN
-F 1 "Screw_Terminal_01x08" H 15130 1701 50  0000 L CNN
-F 2 "Main:Terminal_block_OSTVN08A150" H 15050 1800 50  0001 C CNN
-F 3 "~" H 15050 1800 50  0001 C CNN
-F 4 "On Shore Technology Inc." H 15050 1800 50  0001 C CNN "Manufacturer"
-F 5 "OSTVN08A150" H 15050 1800 50  0001 C CNN "MPN"
-	1    15050 1800
+L Sensor_Humidity:Si7020-A20 U5
+U 1 1 5D9E5346
+P 11000 3000
+F 0 "U5" H 11441 3046 50  0000 L CNN
+F 1 "Si7020-A20" H 11441 2955 50  0000 L CNN
+F 2 "Package_DFN_QFN:DFN-6-1EP_3x3mm_P1mm_EP1.5x2.4mm" H 11000 2600 50  0001 C CNN
+F 3 "https://www.silabs.com/documents/public/data-sheets/Si7020-A20.pdf" H 10800 3300 50  0001 C CNN
+	1    11000 3000
 	1    0    0    -1
 $EndComp
+$Comp
+L Connector:Screw_Terminal_01x03 J3
+U 1 1 5D9E5750
+P 15050 1100
+F 0 "J3" H 15130 1142 50  0000 L CNN
+F 1 "Screw_Terminal_01x03" H 15130 1051 50  0000 L CNN
+F 2 "Main:TerminalBlock_1X3_P5.08mm" H 15050 1100 50  0001 C CNN
+F 3 "~" H 15050 1100 50  0001 C CNN
+F 4 "Phoenix Contact" H 15050 1100 50  0001 C CNN "Manufacturer"
+F 5 "1715734" H 15050 1100 50  0001 C CNN "MPN"
+	1    15050 1100
+	1    0    0    -1
+$EndComp
+$Comp
+L Connector:Screw_Terminal_01x10 J1
+U 1 1 5D9E7CDE
+P 15050 1950
+F 0 "J1" H 15130 1942 50  0000 L CNN
+F 1 "Screw_Terminal_01x10" H 15130 1851 50  0000 L CNN
+F 2 "Main:Terminal_block_OSTVN10A150" H 15050 1950 50  0001 C CNN
+F 3 "~" H 15050 1950 50  0001 C CNN
+F 4 "On Shore Technology Inc." H 15050 1950 50  0001 C CNN "Manufacturer"
+F 5 "OSTVN10A150" H 15050 1950 50  0001 C CNN "MPN"
+	1    15050 1950
+	1    0    0    -1
+$EndComp
+$Comp
+L Connector:Conn_01x01_Male J?
+U 1 1 5D9E855A
+P 15050 4250
+F 0 "J?" H 15023 4273 50  0000 R CNN
+F 1 "Conn_01x01_Male" H 15023 4182 50  0000 R CNN
+F 2 "" H 15050 4250 50  0001 C CNN
+F 3 "~" H 15050 4250 50  0001 C CNN
+	1    15050 4250
+	-1   0    0    -1
+$EndComp
+$Comp
+L Connector:Conn_01x01_Male J?
+U 1 1 5D9E87D0
+P 15050 4450
+F 0 "J?" H 15023 4473 50  0000 R CNN
+F 1 "Conn_01x01_Male" H 15023 4382 50  0000 R CNN
+F 2 "" H 15050 4450 50  0001 C CNN
+F 3 "~" H 15050 4450 50  0001 C CNN
+	1    15050 4450
+	-1   0    0    -1
+$EndComp
 $EndSCHEMATC

Commit message: wip
Parts:
- added J10, J11, J5: Conn_01x03_Male, Main:SOCKET254P-01X03-0705530002, symbol Connector:Conn_01x03_Male
- added J8, J9: Conn_01x01_Male, symbol Connector:Conn_01x01_Male
- J6: renamed from J?; footprint (none) -> Connector_PinHeader_1.00mm:PinHeader_1x01_P1.00mm_Vertical
- gave numbers to parts that had none: 1
Other:
- note added: "Honeywell UART Connector"
- note added: "INPUT POWER"
- note added: "IO Connector"
- note added: "Pogo pins"
- note added: "Temp1"
- note added: "Temp2"
- note added: "UART0"
Changed lines of the file:
@@
 $EndComp
 $Comp
-L Connector:Conn_01x01_Male J?
+L Connector:Conn_01x01_Male J6
 U 1 1 5D9E855A
 P 15050 4250
-F 0 "J?" H 15023 4273 50  0000 R CNN
+F 0 "J6" H 15023 4273 50  0000 R CNN
 F 1 "Conn_01x01_Male" H 15023 4182 50  0000 R CNN
-F 2 "" H 15050 4250 50  0001 C CNN
+F 2 "Connector_PinHeader_1.00mm:PinHeader_1x01_P1.00mm_Vertical" H 15050 4250 50  0001 C CNN
 F 3 "~" H 15050 4250 50  0001 C CNN
 	1    15050 4250
@@
 $EndComp
 $Comp
-L Connector:Conn_01x01_Male J?
+L Connector:Conn_01x01_Male J7
 U 1 1 5D9E87D0
 P 15050 4450
-F 0 "J?" H 15023 4473 50  0000 R CNN
+F 0 "J7" H 15023 4473 50  0000 R CNN
 F 1 "Conn_01x01_Male" H 15023 4382 50  0000 R CNN
 F 2 "" H 15050 4450 50  0001 C CNN
@@
 	-1   0    0    -1
 $EndComp
+Text Notes 14100 1150 0    60   ~ 0
+INPUT POWER
+Text Notes 14150 2000 0    60   ~ 0
+IO Connector
+Text Notes 13450 3350 0    60   ~ 0
+Honeywell UART Connector
+$Comp
+L Connector:Conn_01x01_Male J8
+U 1 1 5D9E8EE7
+P 15050 4650
+F 0 "J8" H 15023 4673 50  0000 R CNN
+F 1 "Conn_01x01_Male" H 15023 4582 50  0000 R CNN
+F 2 "" H 15050 4650 50  0001 C CNN
+F 3 "~" H 15050 4650 50  0001 C CNN
+	1    15050 4650
+	-1   0    0    -1
+$EndComp
+$Comp
+L Connector:Conn_01x01_Male J9
+U 1 1 5D9E8F21
+P 15050 4850
+F 0 "J9" H 15023 4873 50  0000 R CNN
+F 1 "Conn_01x01_Male" H 15023 4782 50  0000 R CNN
+F 2 "" H 15050 4850 50  0001 C CNN
+F 3 "~" H 15050 4850 50  0001 C CNN
+	1    15050 4850
+	-1   0    0    -1
+$EndComp
+Text Notes 14300 4600 0    60   ~ 0
+Pogo pins
+$Comp
+L Connector:Conn_01x03_Male J5
+U 1 1 5D9E9EDD
+P 15050 5500
+F 0 "J5" H 15023 5523 50  0000 R CNN
+F 1 "Conn_01x03_Male" H 15023 5432 50  0000 R CNN
+F 2 "Main:SOCKET254P-01X03-0705530002" H 15050 5500 50  0001 C CNN
+F 3 "~" H 15050 5500 50  0001 C CNN
+F 4 "Molex" H 15050 5500 50  0001 C CNN "Manufacturer"
+F 5 "0705530002" H 15050 5500 50  0001 C CNN "MPN"
+	1    15050 5500
+	-1   0    0    -1
+$EndComp
+$Comp
+L Connector:Conn_01x03_Male J10
+U 1 1 5D9EA090
+P 15050 5900
+F 0 "J10" H 15023 5923 50  0000 R CNN
+F 1 "Conn_01x03_Male" H 15023 5832 50  0000 R CNN
+F 2 "Main:SOCKET254P-01X03-0705530002" H 15050 5900 50  0001 C CNN
+F 3 "~" H 15050 5900 50  0001 C CNN
+F 4 "Molex" H 15050 5900 50  0001 C CNN "Manufacturer"
+F 5 "0705530002" H 15050 5900 50  0001 C CNN "MPN"
+	1    15050 5900
+	-1   0    0    -1
+$EndComp
+Text Notes 14250 5500 0    60   ~ 0
+Temp1
+Text Notes 14250 5900 0    60   ~ 0
+Temp2
+$Comp
+L Connector:Conn_01x03_Male J11
+U 1 1 5D9EA692
+P 15050 6350
+F 0 "J11" H 15023 6373 50  0000 R CNN
+F 1 "Conn_01x03_Male" H 15023 6282 50  0000 R CNN
+F 2 "Main:SOCKET254P-01X03-0705530002" H 15050 6350 50  0001 C CNN
+F 3 "~" H 15050 6350 50  0001 C CNN
+F 4 "Molex" H 15050 6350 50  0001 C CNN "Manufacturer"
+F 5 "0705530002" H 15050 6350 50  0001 C CNN "MPN"
+	1    15050 6350
+	-1   0    0    -1
+$EndComp
+Text Notes 14250 6400 0    60   ~ 0
+UART0
 $EndSCHEMATC

Commit message: wip
Parts:
- added J12: Conn_01x02_Male, Main:AC_terminal_4300.0104, symbol Connector:Conn_01x02_Male
Changed lines of the file:
@@
 Text Notes 14250 6400 0    60   ~ 0
 UART0
+$Comp
+L Connector:Conn_01x02_Male J12
+U 1 1 5D9F81B3
+P 13150 1350
+F 0 "J12" H 13256 1528 50  0000 C CNN
+F 1 "Conn_01x02_Male" H 13256 1437 50  0000 C CNN
+F 2 "Main:AC_terminal_4300.0104" H 13150 1350 50  0001 C CNN
+F 3 "~" H 13150 1350 50  0001 C CNN
+F 4 "Schurter Inc." H 13150 1350 50  0001 C CNN "Manufacturer"
+F 5 "4300.0104" H 13150 1350 50  0001 C CNN "MPN"
+	1    13150 1350
+	1    0    0    -1
+$EndComp
 $EndSCHEMATC

Commit message: wip, needs routing
Parts:
- removed J3: Screw_Terminal_01x03, Main:TerminalBlock_1X3_P5.08mm, symbol Connector:Screw_Terminal_01x03
- added J3: Screw_Terminal_01x02, Main:TerminalBlock_1X2_P5.08mm, symbol Connector:Screw_Terminal_01x02
- J6: footprint Connector_PinHeader_1.00mm:PinHeader_1x01_P1.00mm_Vertical -> Main:POGOPIN_5mm_P70-2300045R; MPN (none) -> P70-2300045R; Manufacturer (none) -> Harwin Inc.
- J7, J8, J9: footprint (none) -> Main:POGOPIN_5mm_P70-2300045R; MPN (none) -> P70-2300045R; Manufacturer (none) -> Harwin Inc.
Changed lines of the file:
@@
-$EndComp
-$Comp
-L Connector:Screw_Terminal_01x03 J3
-U 1 1 5D9E5750
-P 15050 1100
-F 0 "J3" H 15130 1142 50  0000 L CNN
-F 1 "Screw_Terminal_01x03" H 15130 1051 50  0000 L CNN
-F 2 "Main:TerminalBlock_1X3_P5.08mm" H 15050 1100 50  0001 C CNN
-F 3 "~" H 15050 1100 50  0001 C CNN
-F 4 "Phoenix Contact" H 15050 1100 50  0001 C CNN "Manufacturer"
-F 5 "1715734" H 15050 1100 50  0001 C CNN "MPN"
-	1    15050 1100
-	1    0    0    -1
 $EndComp
 $Comp
@@
 F 0 "J6" H 15023 4273 50  0000 R CNN
 F 1 "Conn_01x01_Male" H 15023 4182 50  0000 R CNN
-F 2 "Connector_PinHeader_1.00mm:PinHeader_1x01_P1.00mm_Vertical" H 15050 4250 50  0001 C CNN
+F 2 "Main:POGOPIN_5mm_P70-2300045R" H 15050 4250 50  0001 C CNN
 F 3 "~" H 15050 4250 50  0001 C CNN
+F 4 "Harwin Inc." H 15050 4250 50  0001 C CNN "Manufacturer"
+F 5 "P70-2300045R" H 15050 4250 50  0001 C CNN "MPN"
 	1    15050 4250
-	-1   0    0    -1
-$EndComp
-$Comp
-L Connector:Conn_01x01_Male J7
-U 1 1 5D9E87D0
-P 15050 4450
-F 0 "J7" H 15023 4473 50  0000 R CNN
-F 1 "Conn_01x01_Male" H 15023 4382 50  0000 R CNN
-F 2 "" H 15050 4450 50  0001 C CNN
-F 3 "~" H 15050 4450 50  0001 C CNN
-	1    15050 4450
 	-1   0    0    -1
 $EndComp
@@
 Text Notes 13450 3350 0    60   ~ 0
 Honeywell UART Connector
-$Comp
-L Connector:Conn_01x01_Male J8
-U 1 1 5D9E8EE7
-P 15050 4650
-F 0 "J8" H 15023 4673 50  0000 R CNN
-F 1 "Conn_01x01_Male" H 15023 4582 50  0000 R CNN
-F 2 "" H 15050 4650 50  0001 C CNN
-F 3 "~" H 15050 4650 50  0001 C CNN
-	1    15050 4650
-	-1   0    0    -1
-$EndComp
-$Comp
-L Connector:Conn_01x01_Male J9
-U 1 1 5D9E8F21
-P 15050 4850
-F 0 "J9" H 15023 4873 50  0000 R CNN
-F 1 "Conn_01x01_Male" H 15023 4782 50  0000 R CNN
-F 2 "" H 15050 4850 50  0001 C CNN
-F 3 "~" H 15050 4850 50  0001 C CNN
-	1    15050 4850
-	-1   0    0    -1
-$EndComp
 Text Notes 14300 4600 0    60   ~ 0
 Pogo pins
@@
 	1    0    0    -1
 $EndComp
+$Comp
+L Connector:Screw_Terminal_01x02 J3
+U 1 1 5DA00852
+P 15050 1050
+F 0 "J3" H 15130 1042 50  0000 L CNN
+F 1 "Screw_Terminal_01x02" H 15130 951 50  0000 L CNN
+F 2 "Main:TerminalBlock_1X2_P5.08mm" H 15050 1050 50  0001 C CNN
+F 3 "~" H 15050 1050 50  0001 C CNN
+F 4 "Phoenix Contact" H 15050 1050 50  0001 C CNN "Manufacturer"
+F 5 "1715721" H 15050 1050 50  0001 C CNN "MPN"
+	1    15050 1050
+	1    0    0    -1
+$EndComp
+$Comp
+L Connector:Conn_01x01_Male J7
+U 1 1 5DA01EA6
+P 15050 4450
+F 0 "J7" H 15023 4473 50  0000 R CNN
+F 1 "Conn_01x01_Male" H 15023 4382 50  0000 R CNN
+F 2 "Main:POGOPIN_5mm_P70-2300045R" H 15050 4450 50  0001 C CNN
+F 3 "~" H 15050 4450 50  0001 C CNN
+F 4 "Harwin Inc." H 15050 4450 50  0001 C CNN "Manufacturer"
+F 5 "P70-2300045R" H 15050 4450 50  0001 C CNN "MPN"
+	1    15050 4450
+	-1   0    0    -1
+$EndComp
+$Comp
+L Connector:Conn_01x01_Male J8
+U 1 1 5DA01EE6
+P 15050 4650
+F 0 "J8" H 15023 4673 50  0000 R CNN
+F 1 "Conn_01x01_Male" H 15023 4582 50  0000 R CNN
+F 2 "Main:POGOPIN_5mm_P70-2300045R" H 15050 4650 50  0001 C CNN
+F 3 "~" H 15050 4650 50  0001 C CNN
+F 4 "Harwin Inc." H 15050 4650 50  0001 C CNN "Manufacturer"
+F 5 "P70-2300045R" H 15050 4650 50  0001 C CNN "MPN"
+	1    15050 4650
+	-1   0    0    -1
+$EndComp
+$Comp
+L Connector:Conn_01x01_Male J9
+U 1 1 5DA01F28
+P 15050 4850
+F 0 "J9" H 15023 4873 50  0000 R CNN
+F 1 "Conn_01x01_Male" H 15023 4782 50  0000 R CNN
+F 2 "Main:POGOPIN_5mm_P70-2300045R" H 15050 4850 50  0001 C CNN
+F 3 "~" H 15050 4850 50  0001 C CNN
+F 4 "Harwin Inc." H 15050 4850 50  0001 C CNN "Manufacturer"
+F 5 "P70-2300045R" H 15050 4850 50  0001 C CNN "MPN"
+	1    15050 4850
+	-1   0    0    -1
+$EndComp
 $EndSCHEMATC
