File: pcb/piweather.sch (KiCad schematic (older format))
At the start: 22 parts, among them J1 Screw_Terminal_01x10, J10 Conn_01x03_Male, J11 Conn_01x03_Male, J12 Conn_01x02_Male, J2 Conn_01x08_Male, J3 Screw_Terminal_01x02, J4 Raspberry_Pi_2_3, J5 Conn_01x03_Male, J6 Conn_01x01_Male, J7 Conn_01x01_Male, J8 Conn_01x01_Male, J9 Conn_01x01_Male, U1 FT2232D, U2 PSK-S5B-5, U3 THVD1500, U4 V78E05-1000-SMT-TR, U5 Si7020-A20

Commit message: wip
Parts:
- added C?: CC0603KRX7R9BB333, Main:CAPC0603, symbol cap_smd:CC0603KRX7R9BB333
- added C? (x3): CC0603KRX7R9BB104, Main:CAPC0603, symbol cap_smd:CC0603KRX7R9BB104
- added C?: CP, Capacitor_SMD:C_1206_3216Metric, symbol Device:CP
- added C? (x2): CC0603JRNPO9BN100, Main:CAPC0603, symbol cap_smd:CC0603JRNPO9BN100
- added FB?: Ferrite_Bead_Small, Main:CAPC0603, symbol Device:Ferrite_Bead_Small
- added R?: RC0603FR-071K5L, Main:RESC0603, symbol res_smd:RC0603FR-071K5L
- added R?: RC0603FR-07475RL, Main:RESC0603, symbol res_smd:RC0603FR-07475RL
- added R?: RC0603FR-0710KL, Main:RESC0603, symbol res_smd:RC0603FR-0710KL
- added Y?: Crystal, Crystal:Crystal_SMD_HC49-SD, symbol Device:Crystal
Connections:
- net labels added: +5V, 3V3OUT, AVCC, GND, USBD_N, USBD_P, VCC_FTDI, XTIN, XTOUT, ~RSTOUT
- wire segments 0 -> 85
- no-connect marks 0 -> 2
Other:
- moved on the sheet: J2, J6, J7, J8, J9, U1, U3

Commit message: wip
Connections:
- net labels added: EEDATA, P2_D, P2_R, P2_~RE, P_DE
Changed lines of the file:
@@
 Wire Wire Line
 	5700 9000 5100 9000
+Text Label 5150 7500 0    39   ~ 0
+P2_D
+Text Label 3050 8600 0    39   ~ 0
+EEDATA
+Text Label 5150 7600 0    39   ~ 0
+P2_R
+Text Label 5150 9000 0    39   ~ 0
+P2_~RE
+Text Label 5150 8400 0    39   ~ 0
+P_DE
 $EndSCHEMATC

Commit message: wip
Parts:
- added C? (x4): CC0603KRX7R9BB104, Main:CAPC0603, symbol cap_smd:CC0603KRX7R9BB104
- added C? (x2): GRM21BR60J476ME15K, Main:CAPC0805, symbol cap_smd_extra:GRM21BR60J476ME15K
- added R? (x2): RC0603FR-0710KL, Main:RESC0603, symbol res_smd:RC0603FR-0710KL
Connections:
- net labels added: +3V3, AC_L, AC_N, IN_24V, P1_RXD, P1_TXD, SCL, SDA, V3V3_P1
- net labels removed: VCC_FTDI
- wire segments 85 -> 177
- no-connect marks 2 -> 27
Other:
- note added: "AC IN"
- note added: "INPUT 24V"
- note removed: "INPUT POWER"
- moved on the sheet: C?, FB?, J10, J11, J12, J2, J3, J4, J5, J6, J7, U2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

Commit message: started passive placement
Parts:
- removed C? (x2): CC0603JRNPO9BN100, Main:CAPC0603, symbol cap_smd:CC0603JRNPO9BN100
- removed Y?: Crystal, Crystal:Crystal_SMD_HC49-SD, symbol Device:Crystal
- added R6: RC0603FR-071ML, Main:RESC0603, symbol res_smd:RC0603FR-071ML
- added Y1: Resonator, Main:RESONTATOR_450X200, symbol Device:Resonator
- gave numbers to parts that had none: 17
Connections:
- net labels added: P0_RXD, P0_TXD, P1_3V3, P1_RXD_HW_TXD, P1_TXD_HW_RXD, VCC_FTDI
- net labels removed: P1_RXD, P1_TXD, V3V3_P1
- wire segments 177 -> 178
Other:
- moved on the sheet: C13, J10, J11, J4, J5, U5

Commit message: wip, more placement
Parts:
- added C1, C2: GRM21BR60J476ME15K, Main:CAPC0805, symbol cap_smd_extra:GRM21BR60J476ME15K
- added L1: L, Inductor_SMD:L_Wuerth_MAPI-3020, symbol Device:L
- added R7: RC0603FR-071ML, Main:RESC0603, symbol res_smd:RC0603FR-071ML
- added R8: RC0603FR-0734KL, Main:RESC0603, symbol res_smd:RC0603FR-0734KL
- added U6: TLV61046ADB, Package_TO_SOT_SMD:SOT-23-6, symbol Regulator_Switching:TLV61046ADB
Connections:
- net +5V: now also C2.1, L1.1, U6.4 (EN), U6.6 (VI)
- net GND: now also C1.2, C2.2, R8.2, U6.2 (GND)
- net FB_DCDC: now reaches R4.2, R5.1, U4.6 (Vadj)
- new net +24V: C1.1, R7.1, U6.5 (VOUT)
- new net FB_BOOST: R7.2, R8.1, U6.3 (FB)
- new net SW_BOOST: L1.2, U6.1 (SW)
Changed lines of the file:
@@
 Text Label 3850 5000 0    39   ~ 0
 VCC_FTDI
+$Comp
+L Regulator_Switching:TLV61046ADB U6
+U 1 1 5DA5A7B7
+P 10550 1900
+F 0 "U6" H 10550 2325 50  0000 C CNN
+F 1 "TLV61046ADB" H 10550 2234 50  0000 C CNN
+F 2 "Package_TO_SOT_SMD:SOT-23-6" H 10600 1750 50  0001 L CIN
+F 3 "http://www.ti.com/lit/ds/symlink/tlv61046a.pdf" H 10550 2000 50  0001 C CNN
+	1    10550 1900
+	1    0    0    -1
+$EndComp
+$Comp
+L power:GND #PWR0133
+U 1 1 5DA5AA01
+P 10550 2300
+F 0 "#PWR0133" H 10550 2050 50  0001 C CNN
+F 1 "GND" H 10555 2127 50  0000 C CNN
+F 2 "" H 10550 2300 50  0001 C CNN
+F 3 "" H 10550 2300 50  0001 C CNN
+	1    10550 2300
+	1    0    0    -1
+$EndComp
+Wire Wire Line
+	10550 2300 10550 2100
+$Comp
+L power:+5V #PWR0134
+U 1 1 5DA62243
+P 10050 1500
+F 0 "#PWR0134" H 10050 1350 50  0001 C CNN
+F 1 "+5V" H 10065 1673 50  0000 C CNN
+F 2 "" H 10050 1500 50  0001 C CNN
+F 3 "" H 10050 1500 50  0001 C CNN
+	1    10050 1500
+	1    0    0    -1
+$EndComp
+Wire Wire Line
+	10050 1500 10050 1700
+Wire Wire Line
+	10050 1900 10250 1900
+Wire Wire Line
+	10250 1700 10200 1700
+Connection ~ 10050 1700
+Wire Wire Line
+	10050 1700 10050 1900
+$Comp
+L cap_smd_extra:GRM21BR60J476ME15K C1
+U 1 1 5DA71B4B
+P 11600 2100
+F 0 "C1" H 11692 2259 50  0000 L CNN
+F 1 "GRM21BR60J476ME15K" H 11692 2195 15  0000 L CNN
+F 2 "Main:CAPC0805" H 11692 2156 20  0000 L CNN
+F 3 "" H 11630 2120 50  0000 C CNN
+F 4 "Murata Electronics North America" H 11692 2123 8   0000 L CNN "Manufacturer"
+F 5 "GRM21BR60J476ME15K" H 11820 2020 12  0001 R CNN "MPN"
+F 6 "STUFF" H 11692 2090 20  0000 L CNN "SKU"
+F 7 "47.0 µF" H 11692 2047 20  0000 L CNN "C"
+F 8 "±20%" H 11692 2004 20  0000 L CNN "Tol"
+F 9 "6.3V" H 11692 1961 20  0000 L CNN "Vmax"
+F 10 "X5R" H 11692 1918 20  0000 L CNN "Type"
+	1    11600 2100
+	1    0    0    -1
+$EndComp
+$Comp
+L Device:L L1
+U 1 1 5DA72689
+P 10550 1250
+F 0 "L1" V 10740 1250 50  0000 C CNN
+F 1 "L" V 10649 1250 50  0000 C CNN
+F 2 "Inductor_SMD:L_Wuerth_MAPI-3020" H 10550 1250 50  0001 C CNN
+F 3 "~" H 10550 1250 50  0001 C CNN
+F 4 "Wurth Electronics Inc." V 10550 1250 50  0001 C CNN "Manufacturer"
+F 5 "74438336100" V 10550 1250 50  0001 C CNN "MPN"
+	1    10550 1250
+	0    -1   -1   0
+$EndComp
+Wire Wire Line
+	10200 1700 10200 1250
+Wire Wire Line
+	10200 1250 10400 1250
+Connection ~ 10200 1700
+Wire Wire Line
+	10200 1700 10050 1700
+Wire Wire Line
+	10850 1700 10900 1700
+Wire Wire Line
+	10900 1700 10900 1250
+Wire Wire Line
+	10900 1250 10700 1250
+Wire Wire Line
+	11600 2000 11600 1800
+Wire Wire Line
+	11600 1800 11150 1800
+Wire Wire Line
+	11150 2000 11150 1800
+Connection ~ 11150 1800
+Wire Wire Line
+	11150 1800 10850 1800
+$Comp
+L power:GND #PWR0135
+U 1 1 5DA9C68F
+P 11150 2800
+F 0 "#PWR0135" H 11150 2550 50  0001 C CNN
+F 1 "GND" H 11155 2627 50  0000 C CNN
+F 2 "" H 11150 2800 50  0001 C CNN
+F 3 "" H 11150 2800 50  0001 C CNN
+	1    11150 2800
+	1    0    0    -1
+$EndComp
+Wire Wire Line
+	11150 2650 11150 2800
+$Comp
+L power:GND #PWR0136
+U 1 1 5DAA5282
+P 11600 2400
+F 0 "#PWR0136" H 11600 2150 50  0001 C CNN
+F 1 "GND" H 11605 2227 50  0000 C CNN
+F 2 "" H 11600 2400 50  0001 C CNN
+F 3 "" H 11600 2400 50  0001 C CNN
+	1    11600 2400
+	1    0    0    -1
+$EndComp
+Wire Wire Line
+	11600 2400 11600 2200
+Wire Wire Line
+	11150 2200 11150 2350
+Wire Wire Line
+	10850 1900 10900 1900
+Wire Wire Line
+	10900 1900 10900 2350
+Wire Wire Line
+	10900 2350 11150 2350
+Connection ~ 11150 2350
+Wire Wire Line
+	11150 2350 11150 2450
+Text Label 8500 2100 0    39   ~ 0
+FB_DCDC
+Text Label 10900 2350 0    39   ~ 0
+FB_BOOST
+$Comp
+L res_smd:RC0603FR-071ML R7
+U 1 1 5DAC0C60
+P 11150 2100
+F 0 "R7" H 11209 2248 50  0000 L CNN
+F 1 "RC0603FR-071ML" H 11209 2184 15  0000 L CNN
+F 2 "Main:RESC0603" H 11250 2025 10  0001 C CNN
+F 3 "" H 11180 2120 50  0000 C CNN
+F 4 "Yageo" H 11209 2138 28  0000 L CNN "Manufacturer"
+F 5 "RC0603FR-071ML" H 11209 2094 12  0000 L CNN "MPN"
+F 6 "STUFF" H 11209 2058 20  0000 L CNN "SKU"
+F 7 "1.00 MΩ" H 11209 2015 20  0000 L CNN "Res"
+F 8 "±1%" H 11209 1972 20  0000 L CNN "Tol"
+F 9 "100 mW" H 11209 1929 20  0000 L CNN "Pwr"
+	1    11150 2100
+	1    0    0    -1
+$EndComp
+$Comp
+L res_smd:RC0603FR-0734KL R8
+U 1 1 5DAC1097
+P 11150 2550
+F 0 "R8" H 11209 2698 50  0000 L CNN
+F 1 "RC0603FR-0734KL" H 11209 2634 15  0000 L CNN
+F 2 "Main:RESC0603" H 11250 2475 10  0001 C CNN
+F 3 "" H 11180 2570 50  0000 C CNN
+F 4 "Yageo" H 11209 2588 28  0000 L CNN "Manufacturer"
+F 5 "RC0603FR-0734KL" H 11209 2544 12  0000 L CNN "MPN"
+F 6 "STUFF" H 11209 2508 20  0000 L CNN "SKU"
+F 7 "34.0 kΩ" H 11209 2465 20  0000 L CNN "Res"
+F 8 "±1%" H 11209 2422 20  0000 L CNN "Tol"
+F 9 "100 mW" H 11209 2379 20  0000 L CNN "Pwr"
+	1    11150 2550
+	1    0    0    -1
+$EndComp
+$Comp
+L power:+24V #PWR0137
+U 1 1 5DAC12FE
+P 11600 1550
+F 0 "#PWR0137" H 11600 1400 50  0001 C CNN
+F 1 "+24V" H 11615 1723 50  0000 C CNN
+F 2 "" H 11600 1550 50  0001 C CNN
+F 3 "" H 11600 1550 50  0001 C CNN
+	1    11600 1550
+	1    0    0    -1
+$EndComp
+Wire Wire Line
+	11600 1550 11600 1800
+Connection ~ 11600 1800
+Text Label 10900 1450 0    39   ~ 0
+SW_BOOST
+$Comp
+L cap_smd_extra:GRM21BR60J476ME15K C2
+U 1 1 5DAD58C0
+P 10050 2200
+F 0 "C2" H 10142 2359 50  0000 L CNN
+F 1 "GRM21BR60J476ME15K" H 10142 2295 15  0000 L CNN
+F 2 "Main:CAPC0805" H 10142 2256 20  0000 L CNN
+F 3 "" H 10080 2220 50  0000 C CNN
+F 4 "Murata Electronics North America" H 10142 2223 8   0000 L CNN "Manufacturer"
+F 5 "GRM21BR60J476ME15K" H 10270 2120 12  0001 R CNN "MPN"
+F 6 "STUFF" H 10142 2190 20  0000 L CNN "SKU"
+F 7 "47.0 µF" H 10142 2147 20  0000 L CNN "C"
+F 8 "±20%" H 10142 2104 20  0000 L CNN "Tol"
+F 9 "6.3V" H 10142 2061 20  0000 L CNN "Vmax"
+F 10 "X5R" H 10142 2018 20  0000 L CNN "Type"
+	1    10050 2200
+	1    0    0    -1
+$EndComp
+Wire Wire Line
+	10050 2100 10050 1900
+Connection ~ 10050 1900
+$Comp
+L power:GND #PWR0138
+U 1 1 5DADF008
+P 10050 2500
+F 0 "#PWR0138" H 10050 2250 50  0001 C CNN
+F 1 "GND" H 10055 2327 50  0000 C CNN
+F 2 "" H 10050 2500 50  0001 C CNN
+F 3 "" H 10050 2500 50  0001 C CNN
+	1    10050 2500
+	1    0    0    -1
+$EndComp
+Wire Wire Line
+	10050 2500 10050 2300
 $EndSCHEMATC

Commit message: updated placement, will start routing
Parts:
- added A1: ART, pluggee:pluggeeLogo, symbol systems:ART
- added A2: ART, pluggee:pluggee-QRNEG-127X127, symbol systems:ART
- added A3: ART, Symbol:KiCad-Logo2_6mm_SilkScreen, symbol systems:ART
- added C14, C15: CC0603KRX7R9BB104, Main:CAPC0603, symbol cap_smd:CC0603KRX7R9BB104
- added Q1, Q2: 2N7002, Package_TO_SOT_SMD:SOT-23, symbol Transistor_FET:2N7002
- added R10, R11, R12, R9: RC0603FR-0730K1L, Main:RESC0603, symbol res_smd:RC0603FR-0730K1L
- added U7: 74HC14, symbol 74xx:74HC14
- added U8: LM339, symbol Comparator:LM339
- J10, J11, J5: footprint Main:SOCKET254P-01X03-0705530002 -> Main:SOCKET200P-01X03-S3B-PH-K-S(LF)(SN); MPN 0705530002 -> S3B-PH-K-S(LF)(SN); Manufacturer Molex -> JST
- J6: MPN P70-2300045R -> P70-2200045R
- J8: MPN P70-2300045R -> P70-2200045
Connections:
- net +24V: now also J1.10 (Pin_10), C15.1, U8.3 (V+)
- net +3V3: now also J10.1 (Pin_1), J5.1 (Pin_1), C14.1, R10.1, R11.1, R9.1, U7.14 (VCC)
- net +5V: no longer C7.1
- net GND: now also J1.3 (Pin_3), J10.3 (Pin_3), J5.3 (Pin_3), C14.2, C15.2, Q1.2 (S), Q2.2 (S), R12.2, U7.1, U7.13, U7.3, U7.5, U7.7 (GND), U8.12 (V-)
- net BCM17_PIN11: now reaches J4.11 (GPIO17)
- net BCM17_PIN11: now also U7.8
- net BCM27: now reaches J4.13 (GPIO27)
- net BCM27: now also U8.7 (+)
- net BCM5_PIN29: now reaches J4.29 (GCLK1/GPIO5)
- net BCM5_PIN29: now also J5.2 (Pin_2)
- net BCM12: now reaches J4.32 (PWM0/GPIO12)
- net BCM12: now also U8.5 (+)
- net BCM13: now reaches J4.33 (PWM1/GPIO13)
- net BCM13: now also U8.11 (+)
- net BCM16: now reaches J4.36 (GPIO16)
- net BCM16: now also U8.9 (+)
- net BCM26_PIN37: now reaches J4.37 (GPIO26)
- net BCM26_PIN37: now also U7.10
- net BCM4_PIN7: now reaches J4.7 (GCLK0/GPIO4)
- net BCM4_PIN7: now also J10.2 (Pin_2)
- net RS485_A: now reaches U3.6 (A)
- net RS485_A: now also J1.1 (Pin_1)
- net RS485_B: now reaches U3.7 (B)
- net RS485_B: now also J1.2 (Pin_2)
- net DI17: now reaches J1.4 (Pin_4)
- net DI17: now also Q1.1 (G)
- net DI26: now reaches J1.5 (Pin_5)
- net DI26: now also Q2.1 (G)
- net DO12: now reaches J1.6 (Pin_6)
- net DO12: now also U8.2
- net DO13: now reaches J1.7 (Pin_7)
- net DO13: now also U8.13
- net DO16: now reaches J1.8 (Pin_8)
- net DO16: now also U8.14
- net DO27: now reaches J1.9 (Pin_9)
- net DO27: now also U8.1
- new net REF3V3: C7.1, R11.2, R12.1, U8.10 (-), U8.4 (-), U8.6 (-), U8.8 (-)
- new net ~BCM17: Q1.3 (D), R9.2, U7.9
- new net ~BCM26: Q2.3 (D), R10.2, U7.11
- no-connect marks 27 -> 47
Other:
- note added: "Art Work"
- moved on the sheet: C1, C10, C12, C13, C2, J1, J10, J11, J12, J3, J4, J5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

Commit message: layout in progress
Parts:
- removed R6: RC0603FR-071ML, Main:RESC0603, symbol res_smd:RC0603FR-071ML
- added R6: RC1206FR-071ML, Main:RESC1206, symbol res_smd:RC1206FR-071ML
Connections:
- net XTIN: now also R6.1
- net XTOUT: now also R6.2
Changed lines of the file:
@@
 Wire Wire Line
 	1400 8000 1500 8000
-$Comp
-L res_smd:RC0603FR-071ML R6
-U 1 1 5DAEA189
-P 2350 8000
-F 0 "R6" H 2409 8148 50  0000 L CNN
-F 1 "RC0603FR-071ML" H 2409 8084 15  0000 L CNN
-F 2 "Main:RESC0603" H 2450 7925 10  0001 C CNN
-F 3 "" H 2380 8020 50  0000 C CNN
-F 4 "Yageo" H 2409 8038 28  0000 L CNN "Manufacturer"
-F 5 "RC0603FR-071ML" H 2409 7994 12  0000 L CNN "MPN"
-F 6 "STUFF" H 2409 7958 20  0000 L CNN "SKU"
-F 7 "1.00 MΩ" H 2409 7915 20  0000 L CNN "Res"
-F 8 "±1%" H 2409 7872 20  0000 L CNN "Tol"
-F 9 "100 mW" H 2409 7829 20  0000 L CNN "Pwr"
-	1    2350 8000
-	1    0    0    -1
-$EndComp
 Wire Wire Line
 	2350 7900 2350 7800
@@
 	1    0    0    -1
 $EndComp
+$Comp
+L res_smd:RC1206FR-071ML R6
+U 1 1 5DBA605D
+P 2350 8000
+F 0 "R6" H 2409 8148 50  0000 L CNN
+F 1 "RC1206FR-071ML" H 2409 8084 15  0000 L CNN
+F 2 "Main:RESC1206" H 2450 7925 10  0001 C CNN
+F 3 "" H 2380 8020 50  0000 C CNN
+F 4 "Yageo" H 2409 8038 28  0000 L CNN "Manufacturer"
+F 5 "RC1206FR-071ML" H 2409 7994 12  0000 L CNN "MPN"
+F 6 "STUFF" H 2409 7958 20  0000 L CNN "SKU"
+F 7 "1.00 MΩ" H 2409 7915 20  0000 L CNN "Res"
+F 8 "±1%" H 2409 7872 20  0000 L CNN "Tol"
+F 9 "250 mW" H 2409 7829 20  0000 L CNN "Pwr"
+	1    2350 8000
+	1    0    0    -1
+$EndComp
